File: kicad/04_SDI_CSI.kicad_sch (KiCad schematic)
At the start: 0 parts

Commit message: Add Antmicro SDI ingest sheet and real SDI playback out.
Import GS2971A+CrossLink into sheet 04, require GS2962A playback path (not input loop), and lock IT6616 HDMI CSI.

Co-authored-by: Cursor <cursoragent@cursor.com>
Parts:
- added C1, C15: C_10u_0603, sdi-mipi-bridge-footprints:C_0603_1608Metric, symbol sdi-mipi-bridge:C_10u_0603
- added C10, C11, C12, C13, C14, C16, C17, C18, C19, C2, C20, C21, C22, C3, C32, C33, C34, C36, C4, C5, C6, C65, C7, C8, C9: C_10n_0402, sdi-mipi-bridge-footprints:C_0402_1005Metric, symbol sdi-mipi-bridge:C_10n_0402
- added C23, C31, C42, C52: C_4u7_0402, sdi-mipi-bridge-footprints:C_0402_1005Metric, symbol sdi-mipi-bridge:C_4u7_0402
- added C24, C25, C26, C28, C29, C30, C35, C45, C47, C55, C56, C62: C_1u_0402, sdi-mipi-bridge-footprints:C_0402_1005Metric, symbol sdi-mipi-bridge:C_1u_0402
- added C27: C_5n6_0402, sdi-mipi-bridge-footprints:C_0402_1005Metric, symbol sdi-mipi-bridge:C_5n6_0402
- added C37, C38: C_2u2_0402, sdi-mipi-bridge-footprints:C_0402_1005Metric, symbol sdi-mipi-bridge:C_2u2_0402
- added C39, C40, C41, C44, C46, C48, C49, C50, C51, C53, C54, C57: C_100n_6V3_0402, sdi-mipi-bridge-footprints:C_0402_1005Metric, symbol sdi-mipi-bridge:C_100n_6V3_0402
- added C43: C_6n2_0603, sdi-mipi-bridge-footprints:C_0603_1608Metric, symbol sdi-mipi-bridge:C_6n2_0603
- added C58: C_33u_0603, sdi-mipi-bridge-footprints:C_0603_1608Metric, symbol sdi-mipi-bridge:C_33u_0603
- added C59, C60: C_16p_0402, sdi-mipi-bridge-footprints:C_0402_1005Metric, symbol sdi-mipi-bridge:C_16p_0402
- added C61, C64: C_470n_0402, sdi-mipi-bridge-footprints:C_0402_1005Metric, symbol sdi-mipi-bridge:C_470n_0402
- added C63: C_47n_0402, sdi-mipi-bridge-footprints:C_0402_1005Metric, symbol sdi-mipi-bridge:C_47n_0402
- added D1, D2, D4, D5: LED_G_0603_LG_L29K-G2J1-24-Z, sdi-mipi-bridge-footprints:LED_0603_1608Metric_G, symbol sdi-mipi-bridge:LED_G_0603_LG_L29K-G2J1-24-Z
- added FB1, FB2, FB3: BLM18PG121SH1D, sdi-mipi-bridge-footprints:FB_0603_1608Metric, symbol sdi-mipi-bridge:FB_120Z_2A_0603
- added J1, J2: Conn_BNC_031-70526-21, sdi-mipi-bridge-footprints:Conn_BNC_031-70526-21, symbol sdi-mipi-bridge:Conn_BNC_031-70526-21
- added J3: Conn_FFC_68715014522_ONE-SIDE, sdi-mipi-bridge-footprints:WE_68715014522_ONE-SIDE, symbol sdi-mipi-bridge:Conn_FFC_68715014522_ONE-SIDE
- added J4, J6: PinHeader_2x5_P1.27mm_Vertical, sdi-mipi-bridge-footprints:PinHeader_2x5_P1.27mm_Drill0.65mm, symbol sdi-mipi-bridge:PinHeader_2x5_P1.27mm_Drill0.65mm
- added J5: PinHeader_1x4_P1.27mm_Drill.7mm, sdi-mipi-bridge-footprints:PinHeader_1x4_P1.27mm_Drill0.7mm, symbol sdi-mipi-bridge:PinHeader_1x4_P1.27mm_Drill0.7mm
- added N1: antmicro_logo, sdi-mipi-bridge-footprints:antmicro-logo_scaled_20mm, symbol sdi-mipi-bridge:antmicro_logo
- added N2: oshw_logo, sdi-mipi-bridge-footprints:oshw-logo, symbol sdi-mipi-bridge:oshw_logo
- added R1, R2, R3: R_22R_0402, sdi-mipi-bridge-footprints:R_0402_1005Metric, symbol sdi-mipi-bridge:R_22R_0402
- added R100, R101, R102, R103, R104, R106, R107, R108, R109, R110, R111, R65, R66, R68, R75, R76, R77, R78, R79, R80, R81, R83, R84, R97, R98, R99: R_10k_0402, sdi-mipi-bridge-footprints:R_0402_1005Metric, symbol sdi-mipi-bridge:R_10k_0402
- added R105, R21, R22, R23, R24, R25, R26, R31, R32, R34, R37, R38, R39, R40, R41, R42, R43, R67, R69, R70, R71, R72, R73, R74, R82, R89, R90, R91, R92: R_0R_0402, sdi-mipi-bridge-footprints:R_0402_1005Metric, symbol sdi-mipi-bridge:R_0R_0402
- added R17, R18, R19, R20, R27, R28: R_75R_0603, sdi-mipi-bridge-footprints:R_0603_1608Metric, symbol sdi-mipi-bridge:R_75R_0603
- added R29: R_37R4_0402, sdi-mipi-bridge-footprints:R_0402_1005Metric, symbol sdi-mipi-bridge:R_37R4_0402
- added R30: R_105R_0402, sdi-mipi-bridge-footprints:R_0402_1005Metric, symbol sdi-mipi-bridge:R_105R_0402
- added R33, R64, R88, R93: R_100R_0402, sdi-mipi-bridge-footprints:R_0402_1005Metric, symbol sdi-mipi-bridge:R_100R_0402
- added R35, R36, R95: R_4k7_0402, sdi-mipi-bridge-footprints:R_0402_1005Metric, symbol sdi-mipi-bridge:R_4k7_0402
- added R4: R_750R_0402, sdi-mipi-bridge-footprints:R_0402_1005Metric, symbol sdi-mipi-bridge:R_750R_0402
- added R5, R6: R_120k_0402, sdi-mipi-bridge-footprints:R_0402_1005Metric, symbol sdi-mipi-bridge:R_120k_0402
- added R85, R86, R87, R94: R_2k2_0402, sdi-mipi-bridge-footprints:R_0402_1005Metric, symbol sdi-mipi-bridge:R_2k2_0402
- added R96: R_30R_0402, sdi-mipi-bridge-footprints:R_0402_1005Metric, symbol sdi-mipi-bridge:R_30R_0402
- added SW1: SW_SPST_KMR211NGLFS, sdi-mipi-bridge-footprints:SW_SPST_4.2x2.8, symbol sdi-mipi-bridge:SW_SPST_KMR211NGLFS
- added TP1, TP17, TP18, TP19, TP2, TP20, TP21, TP6: TP_1mm_SMD, sdi-mipi-bridge-footprints:Testpoint_smd_1mm, symbol sdi-mipi-bridge:TP_1mm_SMD
- added TP10, TP11, TP12, TP13, TP14, TP15, TP16, TP7, TP8, TP9: TP_0.75mm_SMD, sdi-mipi-bridge-footprints:TP_SMD_0.75mm, symbol sdi-mipi-bridge:TP_0.75mm_SMD
- added U1: MAX8902B, sdi-mipi-bridge-footprints:TDFN-8-1EP_2x2mm_P0.5mm, symbol sdi-mipi-bridge:MAX8902B
- added U2: GS2971A, sdi-mipi-bridge-footprints:BGA100_11x11mm_SEMTECH, symbol sdi-mipi-bridge:GS2971A
- added U3: GS2988, sdi-mipi-bridge-footprints:QFN-16_1EP_4x4mm_P0.65mm, symbol sdi-mipi-bridge:GS2988
- added U4: CrossLink_LIF-MD6000-6JMG80I, sdi-mipi-bridge-footprints:BGA-80_7x7mm_Layout10x10_P0.65mm, symbol sdi-mipi-bridge:CrossLink_LIF-MD6000-6JMG80I
- added U5: SC18IS602BIPW, sdi-mipi-bridge-footprints:TSSOP-16_4.4x5mm_P0.65mm, symbol sdi-mipi-bridge:SC18IS602BIPW
- added Y1: Oscillator_SMD_27MHz_ABM7, sdi-mipi-bridge-footprints:Oscillator_SMD_Abracon_ABM7-2Pin_6x3.5mm, symbol sdi-mipi-bridge:Oscillator_SMD_27MHz_ABM7
Connections:
- net +3V3: now also C1.2, C19.2, C21.2, C24.2, C26.2, FB1.1, J5.1, J6.1, R21.1, R24.1, R25.1, R26.1, R43.1, R92.2, U1.1 (IN), U1.3 (EN), U4.D5 (VCCAUX), U5.12 (V_{DD})
- net CSI1_CK_N: now also J3.10, U4.A8 (DPHY0_CKN)
- net CSI1_CK_P: now also J3.11, U4.B8 (DPHY0_CKP)
- net CSI1_D0_N: now also J3.7, U4.A7 (DPHY0_DN0)
- net CSI1_D0_P: now also J3.8, U4.B7 (DPHY0_DP0)
- net I2C_SCL: now also J6.4, U4.K2 (PB47/PCLKT0_0/USER_SDA)
- net I2C_SDA: now also J6.2, U4.D1 (PB48/PCLKT0_1/USER_SCL)
- new net: C43.2, C55.1, R27.1, R28.1
- new net: C56.1, R29.1
- new net: TP17.1, U2.H6 (XTAL_OUT)
- new net: TP6.1, U1.5 (~{POK})
- new net: R5.2, R6.1, U1.6 (FB)
- new net: C10.1, U1.7 (BYP)
- new net: R3.2, U2.H4 (WCLK)
- new net: R2.2, U2.J4 (ACLK)
- new net: R1.2, U2.K4 (AMCLK)
- new net: R72.1, U5.14 (A0)
- new net: R73.1, U5.15 (A1)
- new net: R74.1, U5.16 (A2)
- new net: R43.2, U5.3 (~{RESET})
- new net: D2.1, R88.1
- new net: C43.1, J2.1, R27.2
- new net: C27.1, R17.1, R19.1, U3.11 (SDO-)
- new net: C27.2, C31.1, R17.2
- new net: R4.2, U3.4 (RSET)
- new net: R90.2, U4.D2 (VCCPLL_DPHY1), U4.D4 (VCCA_DPHY1)
- new net: R91.2, U4.D7 (VCCPLL_DPHY0), U4.E7 (VCCA_DPHY0)
- new net: R96.2, U4.J1 (PB53/SPI_SCK/MCK/SDA)
- new net: C23.2, R18.1, U3.12 (SDO+)
- new net: TP18.1, U3.14 (~{OSP})
- new net: R71.2, U3.16 (~{EQ_EN})
- new net: D1.1, R33.1
- new net: D4.1, R93.1
- new net: C31.2, J1.1
- new net: R67.2, R85.1, R86.1, R87.1, R94.1
- new net: C23.1, R20.2
- new net: D5.1, R64.1
- new net: J3.47, J3.48, R92.1
- new net: C45.2, R26.2
- new net: R82.2, SW1.2, SW1.4
- new net: U2.B3 (RSV), U2.F2 (RSV)
- new net +1V2: C10.2, C15.2, C2.2, C20.2, C25.2, C39.2, C4.2, C42.2, C48.2, C52.2, C6.2, C8.2, FB2.1, FB3.2, R23.1, R5.1, U1.8 (OUT), U2.D6 (CORE_{VDD}), U2.E6 (CORE_{VDD}), U2.F6 (CORE_{VDD}), U2.G6 (CORE_{VDD}), U4.E4 (VCC), U4.E6 (VCC)
- new net +3.3V: R67.1
- new net +3.3VA: C12.2, C14.2, C17.2, C28.2, C32.2, R21.2, R34.1, U2.B1 (A_{VDD}), U2.E1 (EQ_{VDD}), U2.H1 (BUFF_{VDD})
- new net 20bit_~{10bit}: R80.1, R81.2, U2.H7 (20BIT/~{10BIT}), U4.K8 (PB16C/PCLKT2_1)
- new net AGCN: C61.1, C64.1, U2.G1 (AGC-)
- new net AGCP: C64.2, U2.F1 (AGC+)
- new net AUDIO_MASTER_CLK: J4.10, R1.1
- new net AUDIO_OUTPUT_CH1_2: J4.5, U2.J3 (AOUT_{1/2})
- new net AUDIO_OUTPUT_CH3_4: J4.7, U2.K3 (AOUT_{3/4})
- new net AUDIO_OUTPUT_CH5_6: J4.6, U2.J5 (AOUT_{5/6})
- new net AUDIO_OUTPUT_CH7_8: J4.8, U2.K5 (AOUT_{7/8})
- new net AUDIO_SERIAL_BIT_CLK: J4.1, J4.2, R2.1
- new net AUDIO_WORD_CLK: J4.3, J4.4, R3.1
- new net Audio_EN_~{DIS}: R76.1, R77.2, U2.H3 (AUDIO_EN/~{DIS}), U4.J8 (PB16D/PCLKC2_1)
- new net CDONE: R36.1, R88.2, U4.J2 (PB49/PMU_WKUPN/CDONE)
- new net CRESET_B: J6.8, R35.1, R89.2, U4.H2 (CRESET_B), U5.10 (GPIO2/~{SS2})
- new net CSI1_D1_N: J3.5, U4.A9 (DPHY0_DN1)
- new net CSI1_D1_P: J3.6, U4.B9 (DPHY0_DP1)
- new net CSI1_D2_N: J3.3, U4.A6 (DPHY0_DN2)
- new net CSI1_D2_P: J3.4, U4.B6 (DPHY0_DP2)
- new net CSI1_D3_N: J3.1, U4.A10 (DPHY0_DN3)
- new net CSI1_D3_P: J3.2, U4.B10 (DPHY0_DP3)
- new net D0: TP7.1, U2.K8 (DOUT0)
- new net D1: TP8.1, U2.J8 (DOUT01)
- new net D2: TP9.1, U2.K9 (DOUT02)
- new net D3: TP10.1, U2.K10 (DOUT03)
- new net D4: TP11.1, U2.J9 (DOUT04)
- new net D5: TP12.1, U2.J10 (DOUT05)
- new net D6: TP13.1, U2.H9 (DOUT06)
- new net D7: TP14.1, U2.H10 (DOUT07)
- new net D8: TP15.1, U2.F9 (DOUT08)
- new net D9: TP16.1, U2.F10 (DOUT09)
- new net DOUT10: U2.E9 (DOUT10), U4.J6 (PB29D/PCLKC1_1)
- new net DOUT11: U2.E10 (DOUT11), U4.J5 (PB34D/MIPI_CLKC1_0)
- new net DOUT12: U2.C8 (DOUT12), U4.J4 (PB38D)
- new net DOUT13: U2.C10 (DOUT13), U4.J3 (PB43D)
- new net DOUT14: U2.C9 (DOUT14), U4.E1 (PB34A/GR_PCLK1_0)
- new net DOUT15: U2.B10 (DOUT15), U4.K7 (PB29B/PCLKC1_0)
- new net DOUT16: U2.B9 (DOUT16), U4.K6 (PB29C/PCLKT1_1)
- new net DOUT17: U2.A10 (DOUT17), U4.K5 (PB34C/MIPI_CLKT1_0)
- new net DOUT18: U2.A9 (DOUT18), U4.K4 (PB38C)
- new net DOUT19: U2.B8 (DOUT19), U4.K3 (PB43C)
- new net DVB_ASI: R100.2, R99.1, U2.G8 (DVB_ASI), U4.K10 (PB12C)
- new net F_DE: TP19.1, U2.B5 (STAT2), U4.F9 (PB6A/GR_PCLK2_0)
- new net GNDA: C11.1, C12.1, C13.1, C14.1, C16.1, C17.1, C18.1, C22.1, C28.1, C29.1, C30.1, C32.1, C33.1, C34.1, C36.2, C58.2, C61.2, C62.2, C63.2, C65.2, J1.2, J2.2, J4.9, R100.1, R102.1, R104.1, R107.1, R109.1, R111.1, R20.1, R22.2, R28.2, R29.2, R32.1, R66.1, R75.1, R77.1, R79.1, R81.1, R97.1, R98.1, SW1.1, SW1.3, U2.B4 (VCO_{GND}), U2.C2 (A_{GND}), U2.D2 (A_{GND}), U2.D3 (A_{GND}), U2.D4 (PLL_{GND}), U2.E2 (EQ_{GND}), U2.E3 (A_{GND}), U2.E4 (PLL_{GND}), U2.F3 (A_{GND}), U2.F4 (PLL_{GND}), U2.G2 (A_{GND}), U2.H2 (BUFF_{GND}), U3.10 (SD/~{HD}), U3.17 (EP), U3.3 (V_{EE})
- new net GNDGPLL: C47.1, C51.1, R69.2, U4.G7 (GNDGPLL)
- new net GNDPLL_DPHY: C49.1, C53.1, R70.2, U4.D6 (GNDPLL_DPHY_X)
- new net GNDREF: C1.1, C15.1, C19.1, C2.1, C20.1, C21.1, C24.1, C25.1, C26.1, C3.1, C35.1, C37.1, C38.1, C39.1, C4.1, C40.1, C41.1, C42.1, C44.1, C45.1, C46.1, C48.1, C5.1, C50.1, C52.1, C54.1, C57.1, C59.1, C6.1, C60.1, C7.1, C8.1, C9.1, D1.2, D2.2, D4.2, D5.2, J3.12, J3.15, J3.18, J3.27, J3.30, J3.9, J3.SH, J5.4, J6.10, R22.1, R6.2, R69.1, R70.1, R72.2, R73.2, R74.2, R89.1, U1.2 (GND), U1.4 (GS), U1.9 (EP), U2.B7 (IO_{GND}), U2.D5 (CORE_{GND}), U2.D9 (IO_{GND}), U2.E5 (CORE_{GND}), U2.F5 (CORE_{GND}), U2.G4 (CORE_{GND}), U2.G5 (CORE_{GND}), U2.G9 (IO_{GND}), U2.J7 (IO_{GND}), U4.C1 (GND), U4.C10 (GND), U4.C2 (GNDA_DPHY1), U4.C9 (GNDA_DPHY0), U4.E5 (GND), U4.G2 (GND), U4.G5 (GND), U5.4 (V_{SS})
- new net H_HSYNC: TP1.1, U2.A5 (STAT0), U4.F1 (PB38A)
- new net IOPROC_EN_~{DIS}: R78.1, R79.2, U2.H8 (IOPROC_EN/~{DIS}), U4.H10 (PB2C/MIPI_CLKT2_0)
- new net IO_VDD: C3.2, C35.2, C5.2, C7.2, C9.2, R101.2, R103.2, R106.2, R108.2, R110.2, R25.2, R65.2, R68.2, R76.2, R78.2, R80.2, R83.2, R84.2, R99.2, U2.A7 (IO_{VDD}), U2.D10 (IO_{VDD}), U2.G10 (IO_{VDD}), U2.K7 (IO_{VDD})
- new net JTAG_~{HOST}: R110.1, R111.2, U2.D8 (JTAG/~{HOST}), U4.D9 (PB16A/PCLKT2_0)
- new net LB_CONT: R32.2, R34.2, U2.A3 (LB_CONT)
- new net LF: C63.1, U2.A2 (LF)
- new net LOCKED: R31.1, R33.2, TP20.1, U2.B6 (STAT3)
- new net LOCKED_CL: R31.2, U4.E2 (PB34B)
- new net MIPI1_CLK_N: J3.28, U4.A3 (DPHY1_CKN)
- new net MIPI1_CLK_P: J3.29, U4.B3 (DPHY1_CKP)
- new net MIPI1_D0_N: J3.25, U4.A2 (DPHY1_DN0)
- new net MIPI1_D0_P: J3.26, U4.B2 (DPHY1_DP0)
- new net MIPI1_D1_N: J3.23, U4.A4 (DPHY1_DN1)
- new net MIPI1_D1_P: J3.24, U4.B4 (DPHY1_DP1)
- new net MIPI1_D2_N: J3.21, U4.A1 (DPHY1_DN2)
- new net MIPI1_D2_P: J3.22, U4.B1 (DPHY1_DP2)
- new net MIPI1_D3_N: J3.19, U4.A5 (DPHY1_DN3)
- new net MIPI1_D3_P: J3.20, U4.B5 (DPHY1_DP3)
- new net MISO: J6.7, U4.K1 (PB51/MISO)
- new net MOSI: J6.5, U4.G1 (PB50/MOSI)
- new net PCLK: U2.A8 (PCLK), U4.J7 (PB29A/PCLKT1_0)
- new net RST: J3.33
- new net SCL1: J3.40, R38.1, R40.1
- new net SCL2: J3.42, R42.1
- new net SCLK_TCK: U2.F8 (SCLK_TCK), U5.11 (SCLK)
- new net SCL_GS: J5.3, R40.2, R87.2, U5.8 (SCL)
- new net SDA1: J3.39, R37.1, R39.1
- new net SDA2: J3.41, R41.1
- new net SDA_GS: J5.2, R39.2, R94.2, U5.7 (SDA)
- new net SDIN_TDI: U2.E8 (SDIN_TDI), U5.6 (MOSI)
- new net SDI_N: C56.2, U2.D1 (SDI-)
- new net SDI_P: C55.2, U2.C1 (SDI+)
- new net SDOUT_TDO: U2.E7 (SDOUT_TDO), U5.5 (MISO)
- new net SDO_EN_DIS: R68.1, R75.2, U2.J2 (SDO_EN/DIS), U3.6 (~{DISABLE})
- new net SDO_N: U2.K1 (SDO-), U3.2 (DDI-)
- new net SDO_P: U2.J1 (SDO+), U3.1 (DDI+)
- new net SPI_SCK(SDA): J6.3, R37.2, R41.2, R86.2, R96.1
- new net SPI_SS(SCL): J6.9, R38.2, R42.2, R85.2, R95.1, U4.H1 (PB52/SPI_SS/CSN/SCL)
- new net STANDBY: R108.1, R109.2, U2.K2 (STANDBY), U4.E9 (PB12A/GPLLT2_0)
- new net SW_EN: R101.1, R102.2, U2.D7 (SW_EN), U4.H9 (PB2D/MIPI_CLKC2_0)
- new net TIM_861: R103.1, R104.2, U2.H5 (TIM_861), U4.G9 (PB2A)
- new net USER_LED: R93.2, U4.J10 (PB6C)
- new net USER_SW: R65.1, R66.2, R82.1, U4.J9 (PB6D)
- new net VBG: C62.1, U2.A1 (VBG)
- new net VCCA_DPHY: C38.2, C40.2, C44.2, C49.2, C53.2, FB2.2, R90.1, R91.1
- new net VCCGPLL: C47.2, C51.2, FB3.1, U4.G6 (VCCGPLL)
- new net VCC_IO: C37.2, C41.2, C46.2, C50.2, C54.2, C57.2, FB1.2, R35.2, R36.2, R95.2, U4.F4 (VCCIO0), U4.F5 (VCCIO1), U4.F6 (VCCIO2), U4.F7 (VCCIO2), U4.G4 (VCCIO1)
- new net VCO_VDD: C58.1, R30.2, U2.A4 (VCO_{VDD})
- new net VDD: C18.2, C22.2, C30.2, C34.2, C36.1, C65.1, R18.2, R19.2, R24.2, R4.1, R71.1, U3.9 (V_{CC})
- new net VPP: C11.2, C13.2, C16.2, C29.2, C33.2, R23.2, R30.1, U2.B2 (PLL_{VDD}), U2.C3 (PLL_{VDD}), U2.C4 (PLL_{VDD})
- new net V_VSYNC: TP2.1, U2.A6 (STAT1), U4.F2 (PB38B)
- new net XTAL1: C60.2, U2.K6 (XTAL1), Y1.2
- new net XTAL2: C59.2, U2.J6 (XTAL2), Y1.1
- new net Y_1ANC: TP21.1, U2.C5 (STAT4), U4.F10 (PB6B)
- new net ~{CS}_TMS: U2.F7 (~{CS}_TMS), U5.1 (GPIO0/~{SS0})
- new net ~{DATA_ERROR}: R64.2, U2.C6 (STAT5), U4.E10 (PB12B/GPLLC2_0)
- new net ~{RC_BYP}: R106.1, R107.2, U2.G3 (~{RC_BYP}), U4.G10 (PB2B)
- new net ~{RST_TRST_SOFT}: R105.1, U4.D10 (PB16B/PCLKC2_0)
- new net ~{RST_TRST}: R105.2, R84.1, R98.2, U2.C7 (RESET_TRST)
- new net ~{SMPTE_BYPASS}: R83.1, R97.2, U2.G7 (~{SMPTE_BYPASS}), U4.K9 (PB12D)
- no-connect marks 0 -> 22
Other:
- note added: "CrossLink MIPI transmitter"
- note added: "CrossLink Power Filtering"
- note added: "CrossLink and Semtech at same I2C Line"
- note added: "D10"
- note added: "D11"
- note added: "D12"
- note added: "D13"
- note added: "D14"
- note added: "D15"
- note added: "D16"
- note added: "D17"
- note added: "D18"
- note added: "D19"
- note added: "DEBUG LOOP ONLY: Antmicro J2/GS2988 — product SDI out is sheet 07 (GS2962A playback)"
- note added: "DNP if one I2C used"
- note added: "DPHY0_CLK_N"
- note added: "DPHY0_CLK_P"
- note added: "DPHY0_D0_N"
- note added: "DPHY0_D0_P"
- note added: "DPHY0_D1_N"
- note added: "DPHY0_D1_P"
- note added: "DPHY0_D2_N"
- note added: "DPHY0_D2_P"
- note added: "DPHY0_D3_N"
- note added: "DPHY0_D3_P"
- note added: "DPHY1_CLK_N"
- note added: "DPHY1_CLK_P"
- note added: "DPHY1_D0_N"
- note added: "DPHY1_D0_P"
- note added: "DPHY1_D1_N"
- note added: "DPHY1_D1_P"
- note added: "DPHY1_D2_N"
- note added: "DPHY1_D2_P"
- note added: "DPHY1_D3_N"
- note added: "DPHY1_D3_P"
- note added: "Default configuration resistors"
- note added: "Filtering"
- note added: "GS Power Filtering"
- note added: "GS_I2C"
- note added: "I2C to SPI bridge"
- note added: "I2S connector"
- note added: "LED INDICATORS"
- note added: "LivCast: sheet 04 — Antmicro SDI-MIPI adapted; CSI1 globals to CM5; power from sheet 01"
- note added: "Logotypes"
- note added: "Low noise LDO"
- note added: "MIPI connector"
- note added: "PROTO: J3 FFC OR direct CSI1 to CM5 on carrier"
- note added: "Place close to GS2971A"
- note added: "Power decoupling"
- note added: "Power supply"
- note added: "Programming interace"
- note added: "Pull-up resistors"
- note added: "RESET"
- note added: "SDI deserializer"
- note added: "SDI input"
- note added: "SDI output"
- note added: "Used as RESET button by default"
- note added: "User button"
- note added: "clock"
- note removed: "Global nets (inter-sheet)"
- note removed: "Golden ref: refs/antmicro-sdi-mipi-bridge (openhardware + KiCad PDF)"
- note removed: "J_SDI_IN --> GS2971A --> parallel --> LIF-MD6000-6JMG80I --> CSI1"
- note removed: "Ref: Antmicro sdi-mipi-bridge-hw"
- note removed: "SDI out: GS2962A --> GS2989 --> J_SDI_OUT"
- title: 04 SDI CSI -> 04 SDI CSI — GS2971A + CrossLink (Antmicro-based)
