File: kicad/07_SDI_OUT.kicad_sch (KiCad schematic)
At the start: 0 parts

Commit message: Wire sheet 07 SDI playback path with real symbols.
Add IT66021FN and GS2962A library symbols, TMDS 1:2 buffer to HDMI monitor and SDI out, and expand CM5 HDMI TMDS nets.

Co-authored-by: Cursor <cursoragent@cursor.com>
Parts:
- added J_HDMI_OUT: Conn_HDMI_A, symbol livcast-capture:Conn_HDMI_A
- added J_SDI_OUT: Conn_BNC_031-70526-21, sdi-mipi-bridge-footprints:Conn_BNC_031-70526-21, symbol sdi-mipi-bridge:Conn_BNC_031-70526-21
- added U701: TMDS_BUF_1TO2, symbol livcast-capture:TMDS_BUF_1TO2
- added U702: IT66021FN, symbol livcast-capture:IT66021FN
- added U703: GS2962A, symbol livcast-capture:GS2962A
Connections:
- net GND: now also J_HDMI_OUT.1 (D0_P)
- new net +5V0: J_HDMI_OUT.2 (D0_N)
- new net DE: U703.2 (DIN1)
- new net HDMI_BUF_B_CK_N: U702.14 (I2C_SDA)
- new net HDMI_BUF_B_CK_P: U702.15 (I2C_SCL)
- new net HDMI_BUF_B_D2_N: U702.16 (INT#)
- new net HDMI_MON_CK_N: J_HDMI_OUT.6 (D2_N), U701.13 (OUTA_D0_N)
- new net HDMI_MON_CK_P: J_HDMI_OUT.7 (CK_P), U701.14 (OUTA_D1_P)
- new net HDMI_MON_D0_N: J_HDMI_OUT.12 (+5V), U701.19 (OUTA_CK_N)
- new net HDMI_MON_D0_P: J_HDMI_OUT.13 (GND)
- new net HDMI_MON_D1_N: J_HDMI_OUT.10 (DDC_SCL), U701.17 (OUTA_D2_N)
- new net HDMI_MON_D1_P: J_HDMI_OUT.11 (HPD), U701.18 (OUTA_CK_P)
- new net HDMI_MON_D2_N: J_HDMI_OUT.8 (CK_N), U701.15 (OUTA_D1_N)
- new net HDMI_MON_D2_P: J_HDMI_OUT.9 (DDC_SDA), U701.16 (OUTA_D2_P)
- new net HDMI_TX_CK_N: U701.2 (IN_D0_N)
- new net HDMI_TX_CK_P: U701.3 (IN_D1_P)
- new net HDMI_TX_D0_N: U701.8 (IN_CK_N)
- new net HDMI_TX_D0_P: U701.9 (OE#)
- new net HDMI_TX_D1_N: U701.6 (IN_D2_N)
- new net HDMI_TX_D1_P: U701.7 (IN_CK_P)
- new net HDMI_TX_D2_N: U701.4 (IN_D1_N)
- new net HDMI_TX_D2_P: U701.5 (IN_D2_P)
- new net HS: U703.4 (DIN3)
- new net I2C_SCL: U702.7 (RXC_P)
- new net I2C_SDA: U702.8 (RXC_N)
- new net PCLK: U702.17 (PDATA0), U703.5 (DIN4)
- new net SDI_OUT_P: J_SDI_OUT.1
- new net SDI_TX_SPI_CS: U703.37 (CS#)
- new net VIDEO0: U702.37 (PCLK)
- new net VIDEO1: U702.36 (PDATA19), U703.24 (F_DE)
- new net VIDEO10: U702.27 (PDATA10), U703.15 (DIN14)
- new net VIDEO11: U702.26 (PDATA9), U703.14 (DIN13)
- new net VIDEO12: U702.25 (PDATA8), U703.13 (DIN12)
- new net VIDEO13: U702.24 (PDATA7), U703.12 (DIN11)
- new net VIDEO14: U702.23 (PDATA6), U703.11 (DIN10)
- new net VIDEO15: U702.22 (PDATA5), U703.10 (DIN9)
- new net VIDEO16: U702.21 (PDATA4), U703.9 (DIN8)
- new net VIDEO17: U702.20 (PDATA3), U703.8 (DIN7)
- new net VIDEO18: U702.19 (PDATA2), U703.7 (DIN6)
- new net VIDEO19: U702.18 (PDATA1), U703.6 (DIN5)
- new net VIDEO2: U702.35 (PDATA18), U703.23 (V_VSYNC)
- new net VIDEO3: U702.34 (PDATA17), U703.22 (H_HSYNC)
- new net VIDEO4: U702.33 (PDATA16), U703.21 (PCLK)
- new net VIDEO5: U702.32 (PDATA15), U703.20 (DIN19)
- new net VIDEO6: U702.31 (PDATA14), U703.19 (DIN18)
- new net VIDEO7: U702.30 (PDATA13), U703.18 (DIN17)
- new net VIDEO8: U702.29 (PDATA12), U703.17 (DIN16)
- new net VIDEO9: U702.28 (PDATA11), U703.16 (DIN15)
- new net VS: U703.3 (DIN2)
Other:
- note added: "Decoupling: place per IT66021FN / GS2962A datasheets (not drawn — avoid Device lib dependency)"
- note added: "GS2962A integrated cable driver — GS2989 NOT required on this sheet"
- note added: "GSPI: SDI_TX_SPI_* from CM5 (dedicated CS); I2C_SDA/SCL to IT66021FN"
- note added: "IT66021FN pinout is interface-level (pending full DS/NDA package mapping)"
- note added: "PRODUCT SDI OUT = playback via GS2962A"
- note added: "Path: CM5 HDMI_TX_* --> U701 TMDS 1:2 --> J_HDMI_OUT (monitor) + U702 IT66021FN --> VIDEO[19:0] --> U703 GS2962A --> J_SDI_OUT"
- note added: "Refs U701/U702/U703 avoid clash with sheet 04 Antmicro U1/U2/U3 (functional: buffer / IT66021FN / GS2962A)"
- note added: "Reject: Antmicro J2/GS2988 as product SDI out (see sheet 04 debug only)"
- note added: "SDI out network: SDO --> AC couple + 75R to BNC center; RSET per GS2962 DS; SDO# terminate per DS; shield=GND"
- note removed: "Formats: same as HDMI out program (720p/1080i/1080p); iOS still owns deinterlace for phone path"
- note removed: "GS2962A has integrated cable driver; GS2989 optional if dual drive needed"
- note removed: "Global nets (inter-sheet)"
- note removed: "J_SDI_OUT connector is local to this sheet (product SDI playback BNC)"
- note removed: "Path: CM5 HDMI TX --> ESD/splitter --> IT66021FN (HDMI RX parallel) --> GS2962A --> SDI BNC (J_SDI_OUT)"
- note removed: "REQUIRED: real SDI playback out — NOT SDI-in reclocked loop"
- note removed: "Reject: using Antmicro J2/GS2988 as product SDI out"
