File: kicad/LivCast_Capture.kicad_sch (KiCad schematic)
At the start: 0 parts

Commit message: Add Antmicro SDI ingest sheet and real SDI playback out.
Import GS2971A+CrossLink into sheet 04, require GS2962A playback path (not input loop), and lock IT6616 HDMI CSI.

Co-authored-by: Cursor <cursoragent@cursor.com>
Other:
- added sheet 07 SDI OUT (07_SDI_OUT.kicad_sch)
Changed lines of the file:
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@@
+    )
+  )
+  (sheet
+    (at 25 115)
+    (size 55.88 27.94)
+    (exclude_from_sim no)
+    (in_bom yes)
+    (on_board yes)
+    (dnp no)
+    (fields_autoplaced yes)
+    (stroke (width 0.1524) (type solid))
+    (fill (color 0 0 0 0.0000))
+    (property "Sheetname" "07 SDI OUT" (at 25 114.492 0)
+      (effects (font (size 1.27 1.27)) (justify left bottom))
+    )
+    (property "Sheetfile" "07_SDI_OUT.kicad_sch" (at 25 143.448 0)
+      (effects (font (size 1.27 1.27)) (justify left top))
     )
   )

Commit message: Collapse KiCad design to a single schematic sheet.
Archive hierarchical sheets; keep SDI playback symbols on one A1 overview with Antmicro detail referenced.

Co-authored-by: Cursor <cursoragent@cursor.com>
Parts:
- added J_HDMI_OUT: Conn_HDMI_A, symbol livcast-capture:Conn_HDMI_A
- added J_SDI_OUT: Conn_BNC_031-70526-21, sdi-mipi-bridge-footprints:Conn_BNC_031-70526-21, symbol sdi-mipi-bridge:Conn_BNC_031-70526-21
- added U701: TMDS_BUF_1TO2, symbol livcast-capture:TMDS_BUF_1TO2
- added U702: IT66021FN, symbol livcast-capture:IT66021FN
- added U703: GS2962A, symbol livcast-capture:GS2962A
Connections:
- new net +5V0: J_HDMI_OUT.2 (D0_N)
- new net DE: U703.2 (DIN1)
- new net GND: J_HDMI_OUT.1 (D0_P)
- new net HDMI_BUF_B_CK_N: U702.14 (I2C_SDA)
- new net HDMI_BUF_B_CK_P: U702.15 (I2C_SCL)
- new net HDMI_BUF_B_D2_N: U702.16 (INT#)
- new net HDMI_MON_CK_N: J_HDMI_OUT.6 (D2_N), U701.13 (OUTA_D0_N)
- new net HDMI_MON_CK_P: J_HDMI_OUT.7 (CK_P), U701.14 (OUTA_D1_P)
- new net HDMI_MON_D0_N: J_HDMI_OUT.12 (+5V), U701.19 (OUTA_CK_N)
- new net HDMI_MON_D0_P: J_HDMI_OUT.13 (GND)
- new net HDMI_MON_D1_N: J_HDMI_OUT.10 (DDC_SCL), U701.17 (OUTA_D2_N)
- new net HDMI_MON_D1_P: J_HDMI_OUT.11 (HPD), U701.18 (OUTA_CK_P)
- new net HDMI_MON_D2_N: J_HDMI_OUT.8 (CK_N), U701.15 (OUTA_D1_N)
- new net HDMI_MON_D2_P: J_HDMI_OUT.9 (DDC_SDA), U701.16 (OUTA_D2_P)
- new net HDMI_TX_CK_N: U701.2 (IN_D0_N)
- new net HDMI_TX_CK_P: U701.3 (IN_D1_P)
- new net HDMI_TX_D0_N: U701.8 (IN_CK_N)
- new net HDMI_TX_D0_P: U701.9 (OE#)
- new net HDMI_TX_D1_N: U701.6 (IN_D2_N)
- new net HDMI_TX_D1_P: U701.7 (IN_CK_P)
- new net HDMI_TX_D2_N: U701.4 (IN_D1_N)
- new net HDMI_TX_D2_P: U701.5 (IN_D2_P)
- new net HS: U703.4 (DIN3)
- new net I2C_SCL: U702.7 (RXC_P)
- new net I2C_SDA: U702.8 (RXC_N)
- new net PCLK: U702.17 (PDATA0), U703.5 (DIN4)
- new net SDI_OUT_P: J_SDI_OUT.1
- new net SDI_TX_SPI_CS: U703.37 (CS#)
- new net VIDEO0: U702.37 (PCLK)
- new net VIDEO1: U702.36 (PDATA19), U703.24 (F_DE)
- new net VIDEO10: U702.27 (PDATA10), U703.15 (DIN14)
- new net VIDEO11: U702.26 (PDATA9), U703.14 (DIN13)
- new net VIDEO12: U702.25 (PDATA8), U703.13 (DIN12)
- new net VIDEO13: U702.24 (PDATA7), U703.12 (DIN11)
- new net VIDEO14: U702.23 (PDATA6), U703.11 (DIN10)
- new net VIDEO15: U702.22 (PDATA5), U703.10 (DIN9)
- new net VIDEO16: U702.21 (PDATA4), U703.9 (DIN8)
- new net VIDEO17: U702.20 (PDATA3), U703.8 (DIN7)
- new net VIDEO18: U702.19 (PDATA2), U703.7 (DIN6)
- new net VIDEO19: U702.18 (PDATA1), U703.6 (DIN5)
- new net VIDEO2: U702.35 (PDATA18), U703.23 (V_VSYNC)
- new net VIDEO3: U702.34 (PDATA17), U703.22 (H_HSYNC)
- new net VIDEO4: U702.33 (PDATA16), U703.21 (PCLK)
- new net VIDEO5: U702.32 (PDATA15), U703.20 (DIN19)
- new net VIDEO6: U702.31 (PDATA14), U703.19 (DIN18)
- new net VIDEO7: U702.30 (PDATA13), U703.18 (DIN17)
- new net VIDEO8: U702.29 (PDATA12), U703.17 (DIN16)
- new net VIDEO9: U702.28 (PDATA11), U703.16 (DIN15)
- new net VS: U703.3 (DIN2)
Other:
- removed sheet 01 Power
- removed sheet 02 CM5
- removed sheet 03 HDMI CSI
- removed sheet 04 SDI CSI
- removed sheet 05 USBC Phone
- removed sheet 06 LCD
- removed sheet 07 SDI OUT
- note added: "CM5 HDMI_TX → U701 TMDS_BUF_1TO2 → J_HDMI_OUT + U702 IT66021FN → U703 GS2962A → J_SDI_OUT BNC"
- note added: "CSI0 ← IT6616 (HDMI IN) | CSI1 ← CrossLink (SDI IN) | HDMI_TX → SDI PLAYBACK OUT | USB ← phone gadget"
- note added: "Decoupling: place per IT66021FN / GS2962A datasheets (not drawn — avoid Device lib dependency)"
- note added: "Full detail (do not paste here): refs/antmicro-sdi-mipi-bridge/ + archive_sheets/04_SDI_CSI.kicad_sch"
- note added: "GS2962A integrated cable driver — GS2989 NOT required on this sheet"
- note added: "GSPI: SDI_TX_SPI_* from CM5 (dedicated CS); I2C_SDA/SCL to IT66021FN"
- note added: "IT66021FN pinout is interface-level (pending full DS/NDA package mapping)"
- note added: "J_DTAP (VIN_RAW) | J_USBC_PWR | TPS25751D sink | LM76003 | TPS62130A | OR diodes"
- note added: "J_HDMI_IN → ESD → IT6616 → CSI0_* [IT6616 symbol TBD]"
- note added: "J_LCD — 40-pin Hosyond SPI LCD (local UI). Symbols TBD."
- note added: "J_USBC_PHONE → TPS25751 (source/PD) → TPS25947 (eFuse) → CM5 USB gadget (DP/DN)"
- note added: "LivCast Capture — Complete (single sheet, Rev A)"
- note added: "L→R: POWER → CM5 → HDMI IN / SDI IN → USB / LCD | SDI PLAYBACK OUT (right, real symbols)"
- note added: "Nets: CSI0_* (4lane+ck) | CSI1_* (4lane+ck) | HDMI_TX_* | USB_DP/DN | I2C_* | SPI_* | SDI_TX_SPI_*"
- note added: "No UVC. No internal battery. Antmicro SDI→CSI detail: refs/antmicro-sdi-mipi-bridge + archive_sheets/04_SDI_CSI.kicad_sch"
- note added: "Note: Antmicro J2/GS2988 input-loop is NOT product SDI out — see SDI PLAYBACK OUT (right)."
- note added: "PRODUCT SDI OUT = playback via GS2962A"
- note added: "Path: CM5 HDMI_TX_* --> U701 TMDS 1:2 --> J_HDMI_OUT (monitor) + U702 IT66021FN --> VIDEO[19:0] --> U703 GS2962A --> J_SDI_OUT"
- note added: "Path: HDMI Type-A in → ESD protection → IT6616 HDMI→CSI → CM5 CSI0 (4-lane + clock)"
- note added: "Rails: +5V0, +3V3, +1V8, +1V2, GND | VIN_RAW | PPHV_PD (symbols TBD — power ports below)"
- note added: "Refs U701/U702/U703 avoid clash with sheet 04 Antmicro U1/U2/U3 (functional: buffer / IT66021FN / GS2962A)"
- note added: "Reject: Antmicro J2/GS2988 as product SDI out (see sheet 04 debug only)"
- note added: "SDI IN: J_SDI_IN (BNC) → GS2971A → LIF-MD6000-6JMG80I (CrossLink) → CSI1"
- note added: "SDI out network: SDO --> AC couple + 75R to BNC center; RSET per GS2962 DS; SDO# terminate per DS; shield=GND"
- note added: "U_CM5 (Compute Module 5) — block / footprint TBD"
- note added: "iPhone: USB Ethernet gadget + IP video (not UVC). Symbols TBD."
- note added: "══ REGION CM5 ══"
- note added: "══ REGION HDMI IN ══"
- note added: "══ REGION LCD ══"
- note added: "══ REGION POWER ══"
- note added: "══ REGION SDI IN (Antmicro path — condensed) ══"
- note added: "══ REGION SDI PLAYBACK OUT (from archive 07 — real symbols) ══"
- note added: "══ REGION USB PHONE ══"
- note removed: "LivCast Capture — TOP (Rev A)"
- note removed: "No UVC. No internal battery. iOS handles format."
- note removed: "SDI RX+CrossLink CSI1 | HDMI IT6616 CSI0 | CM5 | USB-C data+charge | D-Tap+USB-C PD"
- company: LivCast / View Vision -> LivCast
- title: LivCast Capture — Top -> LivCast Capture — Complete

Commit message: Fix schematic label overlap with wider pin pitch and IC spacing.
Regenerate CM5/IT66021/GS2962/TMDS symbols at 3.81mm pitch, spread U701–U703 on A0, and realign nets so dense HDMI/CSI/VIDEO labels no longer collide.

Co-authored-by: Cursor <cursoragent@cursor.com>
Parts:
- added J101: Conn_DTAP, symbol livcast-capture:Conn_DTAP
- added J102: Conn_USB_C_PWR, symbol livcast-capture:Conn_USB_C_PWR
- added J501: Conn_USB_C_DATA, symbol livcast-capture:Conn_USB_C_DATA
- added U101, U501: TPS25751D, symbol livcast-capture:TPS25751D
- added U102: LM76003, symbol livcast-capture:LM76003
- added U103: TPS62130A, symbol livcast-capture:TPS62130A
- added U201: CM5, symbol livcast-capture:CM5_IO
Connections:
- net +5V0: now also U201.1 (+5V_1), U201.2 (+5V_2), U201.3 (+5V_3); no longer J_HDMI_OUT.2 (D0_N)
- net DE: now also U702.40 (DE), U703.24 (F_DE); no longer U703.2 (DIN1)
- net GND: now also J101.2 (GND), J102.4 (GND), J501.6 (GND), U101.11 (GND2), U101.4 (GND), U102.3 (GND), U103.3 (GND), U201.4 (GND_1), U201.5 (GND_2), U201.6 (GND_3), U501.11 (GND2), U501.4 (GND); no longer J_HDMI_OUT.1 (D0_P)
- net HDMI_BUF_B_CK_N: now also U701.27 (OUTB_CK_N), U702.8 (RXC_N); no longer U702.14 (I2C_SDA)
- net HDMI_BUF_B_CK_P: now also U701.26 (OUTB_CK_P), U702.7 (RXC_P); no longer U702.15 (I2C_SCL)
- net HDMI_BUF_B_D0_N: now also U701.21 (OUTB_D0_N), U702.2 (RX0_N)
- net HDMI_BUF_B_D0_P: now also U701.20 (OUTB_D0_P), U702.1 (RX0_P)
- net HDMI_BUF_B_D1_N: now also U701.23 (OUTB_D1_N), U702.4 (RX1_N)
- net HDMI_BUF_B_D1_P: now also U701.22 (OUTB_D1_P), U702.3 (RX1_P)
- net HDMI_BUF_B_D2_N: now also U701.25 (OUTB_D2_N), U702.6 (RX2_N); no longer U702.16 (INT#)
- net HDMI_BUF_B_D2_P: now also U701.24 (OUTB_D2_P), U702.5 (RX2_P)
- net HDMI_MON_CK_N: now also J_HDMI_OUT.8 (CK_N), U701.19 (OUTA_CK_N); no longer J_HDMI_OUT.6 (D2_N), U701.13 (OUTA_D0_N)
- net HDMI_MON_CK_P: now also U701.18 (OUTA_CK_P); no longer U701.14 (OUTA_D1_P)
- net HDMI_MON_D0_N: now also J_HDMI_OUT.2 (D0_N), U701.13 (OUTA_D0_N); no longer J_HDMI_OUT.12 (+5V), U701.19 (OUTA_CK_N)
- net HDMI_MON_D0_P: now also J_HDMI_OUT.1 (D0_P), U701.12 (OUTA_D0_P); no longer J_HDMI_OUT.13 (GND)
- net HDMI_MON_D1_N: now also J_HDMI_OUT.4 (D1_N), U701.15 (OUTA_D1_N); no longer J_HDMI_OUT.10 (DDC_SCL), U701.17 (OUTA_D2_N)
- net HDMI_MON_D1_P: now also J_HDMI_OUT.3 (D1_P), U701.14 (OUTA_D1_P); no longer J_HDMI_OUT.11 (HPD), U701.18 (OUTA_CK_P)
- net HDMI_MON_D2_N: now also J_HDMI_OUT.6 (D2_N), U701.17 (OUTA_D2_N); no longer J_HDMI_OUT.8 (CK_N), U701.15 (OUTA_D1_N)
- net HDMI_MON_D2_P: now also J_HDMI_OUT.5 (D2_P); no longer J_HDMI_OUT.9 (DDC_SDA)
- net HDMI_TX_CK_N: now also U701.8 (IN_CK_N), U201.25 (HDMI_TX_CK_N); no longer U701.2 (IN_D0_N)
- net HDMI_TX_CK_P: now also U701.7 (IN_CK_P), U201.24 (HDMI_TX_CK_P); no longer U701.3 (IN_D1_P)
- net HDMI_TX_D0_N: now also U701.2 (IN_D0_N), U201.19 (HDMI_TX_D0_N); no longer U701.8 (IN_CK_N)
- net HDMI_TX_D0_P: now also U701.1 (IN_D0_P), U201.18 (HDMI_TX_D0_P); no longer U701.9 (OE#)
- net HDMI_TX_D1_N: now also U701.4 (IN_D1_N), U201.21 (HDMI_TX_D1_N); no longer U701.6 (IN_D2_N)
- net HDMI_TX_D1_P: now also U701.3 (IN_D1_P), U201.20 (HDMI_TX_D1_P); no longer U701.7 (IN_CK_P)
- net HDMI_TX_D2_N: now also U701.6 (IN_D2_N), U201.23 (HDMI_TX_D2_N); no longer U701.4 (IN_D1_N)
- net HDMI_TX_D2_P: now also U201.22 (HDMI_TX_D2_P)
- net HS: now also U702.38 (HS), U703.22 (H_HSYNC); no longer U703.4 (DIN3)
- net I2C_SCL: now also U101.7 (I2C_SCL), U201.10 (I2C_SCL), U501.7 (I2C_SCL); no longer U702.7 (RXC_P)
- net I2C_SDA: now also U101.6 (I2C_SDA), U201.9 (I2C_SDA), U501.6 (I2C_SDA); no longer U702.8 (RXC_N)
- net PCLK: now also U702.37 (PCLK), U703.21 (PCLK); no longer U702.17 (PDATA0), U703.5 (DIN4)
- net SDI_TX_SPI_CS: now also U201.17 (SDI_TX_SPI_CS)
- net SDI_TX_SPI_MISO: now also U703.35 (SDOUT)
- net SDI_TX_SPI_MOSI: now also U703.34 (SDIN), U201.15 (SDI_TX_SPI_MOSI)
- net SDI_TX_SPI_SCK: now also U703.36 (SCLK), U201.16 (SDI_TX_SPI_SCK)
- net VIDEO0: now also U702.17 (PDATA0), U703.1 (DIN0); no longer U702.37 (PCLK)
- net VIDEO1: now also U702.18 (PDATA1), U703.2 (DIN1); no longer U702.36 (PDATA19), U703.24 (F_DE)
- net VIDEO10: now also U703.11 (DIN10); no longer U703.15 (DIN14)
- net VIDEO11: now also U702.28 (PDATA11), U703.12 (DIN11); no longer U702.26 (PDATA9), U703.14 (DIN13)
- net VIDEO12: now also U702.29 (PDATA12); no longer U702.25 (PDATA8)
- net VIDEO13: now also U702.30 (PDATA13), U703.14 (DIN13); no longer U702.24 (PDATA7), U703.12 (DIN11)
- net VIDEO14: now also U702.31 (PDATA14), U703.15 (DIN14); no longer U702.23 (PDATA6), U703.11 (DIN10)
- net VIDEO15: now also U702.32 (PDATA15), U703.16 (DIN15); no longer U702.22 (PDATA5), U703.10 (DIN9)
- net VIDEO16: now also U702.33 (PDATA16), U703.17 (DIN16); no longer U702.21 (PDATA4), U703.9 (DIN8)
- net VIDEO17: now also U702.34 (PDATA17), U703.18 (DIN17); no longer U702.20 (PDATA3), U703.8 (DIN7)
- net VIDEO18: now also U702.35 (PDATA18), U703.19 (DIN18); no longer U702.19 (PDATA2), U703.7 (DIN6)
- net VIDEO19: now also U702.36 (PDATA19), U703.20 (DIN19); no longer U702.18 (PDATA1), U703.6 (DIN5)
- net VIDEO2: now also U702.19 (PDATA2), U703.3 (DIN2); no longer U702.35 (PDATA18), U703.23 (V_VSYNC)
- net VIDEO3: now also U702.20 (PDATA3), U703.4 (DIN3); no longer U702.34 (PDATA17), U703.22 (H_HSYNC)
- net VIDEO4: now also U702.21 (PDATA4), U703.5 (DIN4); no longer U702.33 (PDATA16), U703.21 (PCLK)
- net VIDEO5: now also U702.22 (PDATA5), U703.6 (DIN5); no longer U702.32 (PDATA15), U703.20 (DIN19)
- net VIDEO6: now also U702.23 (PDATA6), U703.7 (DIN6); no longer U702.31 (PDATA14), U703.19 (DIN18)
- net VIDEO7: now also U702.24 (PDATA7), U703.8 (DIN7); no longer U702.30 (PDATA13), U703.18 (DIN17)
- net VIDEO8: now also U702.25 (PDATA8), U703.9 (DIN8); no longer U702.29 (PDATA12), U703.17 (DIN16)
- net VIDEO9: now also U702.26 (PDATA9), U703.10 (DIN9); no longer U702.28 (PDATA11), U703.16 (DIN15)
- net VS: now also U702.39 (VS), U703.23 (V_VSYNC); no longer U703.3 (DIN2)
- net SDI_OUT_P: no longer names the net of J_SDI_OUT.1
- new net BOOT: U102.9 (BOOT), U103.9 (BOOT)
- new net CC1: J102.2 (CC1), J501.4 (CC1), U101.2 (CC1), U501.2 (CC1)
- new net CC2: J102.3 (CC2), J501.5 (CC2), U101.3 (CC2), U501.3 (CC2)
- new net CSI0_CK_N: U201.35 (CSI0_CK_N)
- new net CSI0_CK_P: U201.34 (CSI0_CK_P)
- new net CSI0_D0_N: U201.27 (CSI0_D0_N)
- new net CSI0_D0_P: U201.26 (CSI0_D0_P)
- new net CSI0_D1_N: U201.29 (CSI0_D1_N)
- new net CSI0_D1_P: U201.28 (CSI0_D1_P)
- new net CSI0_D2_N: U201.31 (CSI0_D2_N)
- new net CSI0_D2_P: U201.30 (CSI0_D2_P)
- new net CSI0_D3_N: U201.33 (CSI0_D3_N)
- new net CSI0_D3_P: U201.32 (CSI0_D3_P)
- new net CSI1_CK_N: U201.45 (CSI1_CK_N)
- new net CSI1_CK_P: U201.44 (CSI1_CK_P)
- new net CSI1_D0_N: U201.37 (CSI1_D0_N)
- new net CSI1_D0_P: U201.36 (CSI1_D0_P)
- new net CSI1_D1_N: U201.39 (CSI1_D1_N)
- new net CSI1_D1_P: U201.38 (CSI1_D1_P)
- new net CSI1_D2_N: U201.41 (CSI1_D2_N)
- new net CSI1_D2_P: U201.40 (CSI1_D2_P)
- new net CSI1_D3_N: U201.43 (CSI1_D3_N)
- new net CSI1_D3_P: U201.42 (CSI1_D3_P)
- new net EN: U102.2 (EN), U103.2 (EN)
- new net FB: U102.4 (FB), U103.4 (FB)
- new net GPIO1: U101.10 (GPIO1), U501.10 (GPIO1)
- new net PG: U102.8 (PG), U103.8 (PG)
- new net PP5V: U101.8 (PP5V), U501.8 (PP5V)
- new net PPHV: U101.9 (PPHV), U501.9 (PPHV)
- new net SPI_CS: U201.14 (SPI_CS)
- new net SPI_MISO: U201.12 (SPI_MISO)
- new net SPI_MOSI: U201.11 (SPI_MOSI)
- new net SPI_SCK: U201.13 (SPI_SCK)
- new net SS: U102.5 (SS), U103.5 (SS)
- new net SW: U102.6 (SW), U103.6 (SW)
- new net USB_DN: J501.3 (USB_DN), U201.8 (USB_DN)
- new net USB_DP: J501.2 (USB_DP), U201.7 (USB_DP)
- new net VBUS: J102.1 (VBUS), J501.1 (VBUS), U101.1 (VBUS), U501.1 (VBUS)
- new net VIN: J101.1 (VIN), U102.1 (VIN), U103.1 (VIN)
- new net VIN_3V3: U101.5 (VIN_3V3), U501.5 (VIN_3V3)
- new net VOUT: U102.7 (VOUT), U103.7 (VOUT)
Other:
- note added: "NET ALIAS: HDMI_TX_* globals; VIDEO[19:0] DE VS HS PCLK locals; HDMI_BUF_B_* HDMI_MON_*"
- note added: "Overlap fix: 3.81mm pitch; U701-U703 spread; A0"
- note added: "REGION POWER / CM5 / USB — see aliases at x=300"
- moved on the sheet: J_HDMI_OUT, J_SDI_OUT, U701, U702, U703

Commit message: Fix schematic layout: wire stubs, VIDEO bus, spaced ICs.
Stop placing net labels on pin bodies; rebuild CM5 and SDI playback region for readability.

Co-authored-by: Cursor <cursoragent@cursor.com>
Parts:
- removed J501: Conn_USB_C_DATA, symbol livcast-capture:Conn_USB_C_DATA
- removed J_HDMI_OUT: Conn_HDMI_A, symbol livcast-capture:Conn_HDMI_A
- removed J_SDI_OUT: Conn_BNC_031-70526-21, sdi-mipi-bridge-footprints:Conn_BNC_031-70526-21, symbol sdi-mipi-bridge:Conn_BNC_031-70526-21
- removed U501: TPS25751D, symbol livcast-capture:TPS25751D
- added J201: Conn_USB_C_DATA, symbol livcast-capture:Conn_USB_C_DATA
- added J701: Conn_HDMI_A, symbol livcast-capture:Conn_HDMI_A
- added J702: Conn_BNC_031-70526-21, symbol sdi-mipi-bridge:Conn_BNC_031-70526-21
- added U202: TPS25751D, symbol livcast-capture:TPS25751D
- U201: value CM5 -> CM5_IO
Connections:
- net PP5V is gone; now on net +5V0: U101.8 (PP5V)
- net PPHV is gone; now on net VIN_RAW: U101.9 (PPHV)
- net VIN_3V3 is gone; now on net +3V3: U101.5 (VIN_3V3)
- net +1V2: now also U702.43 (VDD12), U703.38 (VDD_CORE_1V2), U703.41 (VDD_CD)
- net +1V8: now also U702.42 (VDD18)
- net +3V3: now also U103.7 (VOUT), U701.10 (VDD), U702.41 (VDD33), U703.27 (SDO_EN), U703.28 (STANDBY#), U703.29 (BIT20_10), U703.32 (SMPTE_BYPASS), U703.39 (VDD_IO), U703.40 (VDD_A_3V3), U202.5 (VIN_3V3)
- net +5V0: now also U102.7 (VOUT), U103.1 (VIN), U702.12 (+5V_HDMI), J701.12 (+5V), U202.8 (PP5V)
- net GND: now also U701.11 (GND), U702.44 (GND1), U702.45 (GND2), U702.46 (GND3), U703.30 (RATE_SEL0), U703.31 (RATE_SEL1), U703.33 (DVB_ASI), U703.42 (GND1), U703.43 (GND2), U703.44 (GND3), U703.45 (GND4), J201.6 (GND), J701.13 (GND), J701.14 (SHIELD), J702.2, U202.11 (GND2), U202.4 (GND)
- net I2C_SCL: now also U702.15 (I2C_SCL), U202.7 (I2C_SCL)
- net I2C_SDA: now also U702.14 (I2C_SDA), U202.6 (I2C_SDA)
- net USB_DN: now also J201.3 (USB_DN)
- net USB_DP: now also J201.2 (USB_DP)
- net VIN_RAW: now also J101.1 (VIN), U102.1 (VIN), U202.9 (PPHV)
- net DDC_SDA: now reaches U702.10 (DDC_SDA)
- net DDC_SDA: now also J701.9 (DDC_SDA)
- net DDC_SCL: now reaches U702.11 (DDC_SCL)
- net DDC_SCL: now also J701.10 (DDC_SCL)
- net IT_RESET_N: now reaches U702.13 (RESET#)
- net IT_INT_N: now reaches U702.16 (INT#)
- net HPD_IT: now reaches U702.9 (HPD)
- net OE_N: now reaches U701.9 (OE#)
- net SDI_TX_P: now reaches U703.25 (SDO)
- net SDI_TX_P: now also J702.1
- net SDI_TX_N: now reaches U703.26 (SDO#)
- net BOOT renamed BOOT_3V3
- net BOOT_3V3: no longer U102.9 (BOOT)
- net CC1 renamed CC1_IN
- net CC2 renamed CC2_IN
- net EN renamed +3V3_EN
- net +3V3_EN: no longer U102.2 (EN)
- net FB renamed FB_3V3
- net FB_3V3: no longer U102.4 (FB)
- net GPIO1 renamed PD_GPIO1
- net HDMI_BUF_B_CK_N renamed HDMI_RX_CK_N
- net HDMI_BUF_B_CK_P renamed HDMI_RX_CK_P
- net HDMI_BUF_B_D0_N renamed HDMI_RX_D0_N
- net HDMI_BUF_B_D0_P renamed HDMI_RX_D0_P
- net HDMI_BUF_B_D1_N renamed HDMI_RX_D1_N
- net HDMI_BUF_B_D1_P renamed HDMI_RX_D1_P
- net HDMI_BUF_B_D2_N renamed HDMI_RX_D2_N
- net HDMI_BUF_B_D2_P renamed HDMI_RX_D2_P
- net HDMI_MON_CK_N renamed HDMI_OUT_CK_N
- net HDMI_OUT_CK_N: now also J701.8 (CK_N)
- net HDMI_MON_CK_P renamed HDMI_OUT_CK_P
- net HDMI_OUT_CK_P: now also J701.7 (CK_P)
- net HDMI_MON_D0_N renamed HDMI_OUT_D0_N
- net HDMI_OUT_D0_N: now also J701.2 (D0_N)
- net HDMI_MON_D0_P renamed HDMI_OUT_D0_P
- net HDMI_OUT_D0_P: now also J701.1 (D0_P)
- net HDMI_MON_D1_N renamed HDMI_OUT_D1_N
- net HDMI_OUT_D1_N: now also J701.4 (D1_N)
- net HDMI_MON_D1_P renamed HDMI_OUT_D1_P
- net HDMI_OUT_D1_P: now also J701.3 (D1_P)
- net HDMI_MON_D2_N renamed HDMI_OUT_D2_N
- net HDMI_OUT_D2_N: now also J701.6 (D2_N)
- net HDMI_MON_D2_P renamed HDMI_OUT_D2_P
- net HDMI_OUT_D2_P: now also J701.5 (D2_P)
- net PG renamed PG_3V3
- net PG_3V3: no longer U102.8 (PG)
- net SDI_TX_SPI_MISO renamed SPI_MISO_GS
- net SS renamed SS_3V3
- net SS_3V3: no longer U102.5 (SS)
- net SW renamed SW_3V3
- net SW_3V3: no longer U102.6 (SW)
- net VBUS renamed VBUS_IN
- removed net VIN: J101.1 (VIN), U102.1 (VIN), U103.1 (VIN)
- removed net VOUT: U102.7 (VOUT), U103.7 (VOUT)
- new net +5V_EN: U102.2 (EN)
- new net BOOT_5V: U102.9 (BOOT)
- new net CC1_PHONE: J201.4 (CC1), U202.2 (CC1)
- new net CC2_PHONE: J201.5 (CC2), U202.3 (CC2)
- new net FB_5V: U102.4 (FB)
- new net HPD_OUT: J701.11 (HPD)
- new net PD_SRC_GPIO: U202.10 (GPIO1)
- new net PG_5V: U102.8 (PG)
- new net SS_5V: U102.5 (SS)
- new net SW_5V: U102.6 (SW)
- new net VBUS_PHONE: J201.1 (VBUS), U202.1 (VBUS)
Other:
- note added: "CM5 I/O"
- note added: "HDMI IN ingest - TBD (archive_sheets/03)"
- note added: "HDMI OUT (monitor)"
- note added: "HDMI TMDS (CM5 -> buffer)"
- note added: "HDMI to IT66021FN"
- note added: "LCD / DSI - TBD (archive_sheets/06)"
- note added: "LivCast Capture - Complete (single sheet, Rev A)"
- note added: "POWER"
- note added: "Power column left. Labels on wire stubs >=10mm from pins. Ingest TBD: archive_sheets + README.md"
- note added: "Rails"
- note added: "Rule: never place net labels on pin bodies."
- note added: "SDI IN ingest - TBD (archive_sheets/04, Antmicro)"
- note added: "SDI OUT"
- note added: "SDI playback: CM5 HDMI TX -> TMDS 1:2 -> HDMI mon + IT66021FN -> VIDEO[19:0] bus -> GS2962A -> BNC"
- note added: "USB-C phone (network video)"
- note added: "VIDEO[19:0] parallel bus"
- note removed: "CM5 HDMI_TX → U701 TMDS_BUF_1TO2 → J_HDMI_OUT + U702 IT66021FN → U703 GS2962A → J_SDI_OUT BNC"
- note removed: "CSI0 ← IT6616 (HDMI IN) | CSI1 ← CrossLink (SDI IN) | HDMI_TX → SDI PLAYBACK OUT | USB ← phone gadget"
- note removed: "Decoupling: place per IT66021FN / GS2962A datasheets (not drawn — avoid Device lib dependency)"
- note removed: "Full detail (do not paste here): refs/antmicro-sdi-mipi-bridge/ + archive_sheets/04_SDI_CSI.kicad_sch"
- note removed: "GS2962A integrated cable driver — GS2989 NOT required on this sheet"
- note removed: "GSPI: SDI_TX_SPI_* from CM5 (dedicated CS); I2C_SDA/SCL to IT66021FN"
- note removed: "IT66021FN pinout is interface-level (pending full DS/NDA package mapping)"
- note removed: "J_DTAP (VIN_RAW) | J_USBC_PWR | TPS25751D sink | LM76003 | TPS62130A | OR diodes"
- note removed: "J_HDMI_IN → ESD → IT6616 → CSI0_* [IT6616 symbol TBD]"
- note removed: "J_LCD — 40-pin Hosyond SPI LCD (local UI). Symbols TBD."
- note removed: "J_USBC_PHONE → TPS25751 (source/PD) → TPS25947 (eFuse) → CM5 USB gadget (DP/DN)"
- note removed: "LivCast Capture — Complete (single sheet, Rev A)"
- note removed: "L→R: POWER → CM5 → HDMI IN / SDI IN → USB / LCD | SDI PLAYBACK OUT (right, real symbols)"
- note removed: "NET ALIAS: HDMI_TX_* globals; VIDEO[19:0] DE VS HS PCLK locals; HDMI_BUF_B_* HDMI_MON_*"
- note removed: "Nets: CSI0_* (4lane+ck) | CSI1_* (4lane+ck) | HDMI_TX_* | USB_DP/DN | I2C_* | SPI_* | SDI_TX_SPI_*"
- note removed: "No UVC. No internal battery. Antmicro SDI→CSI detail: refs/antmicro-sdi-mipi-bridge + archive_sheets/04_SDI_CSI.kicad_sch"
- note removed: "Note: Antmicro J2/GS2988 input-loop is NOT product SDI out — see SDI PLAYBACK OUT (right)."
- note removed: "Overlap fix: 3.81mm pitch; U701-U703 spread; A0"
- note removed: "PRODUCT SDI OUT = playback via GS2962A"
- note removed: "Path: CM5 HDMI_TX_* --> U701 TMDS 1:2 --> J_HDMI_OUT (monitor) + U702 IT66021FN --> VIDEO[19:0] --> U703 GS2962A --> J_SDI_OUT"
- note removed: "Path: HDMI Type-A in → ESD protection → IT6616 HDMI→CSI → CM5 CSI0 (4-lane + clock)"
- note removed: "REGION POWER / CM5 / USB — see aliases at x=300"
- note removed: "Rails: +5V0, +3V3, +1V8, +1V2, GND | VIN_RAW | PPHV_PD (symbols TBD — power ports below)"
- note removed: "Refs U701/U702/U703 avoid clash with sheet 04 Antmicro U1/U2/U3 (functional: buffer / IT66021FN / GS2962A)"
- note removed: "Reject: Antmicro J2/GS2988 as product SDI out (see sheet 04 debug only)"
- note removed: "SDI IN: J_SDI_IN (BNC) → GS2971A → LIF-MD6000-6JMG80I (CrossLink) → CSI1"
- note removed: "SDI out network: SDO --> AC couple + 75R to BNC center; RSET per GS2962 DS; SDO# terminate per DS; shield=GND"
- note removed: "U_CM5 (Compute Module 5) — block / footprint TBD"
- note removed: "iPhone: USB Ethernet gadget + IP video (not UVC). Symbols TBD."
- note removed: "══ REGION CM5 ══"
- note removed: "══ REGION HDMI IN ══"
- note removed: "══ REGION LCD ══"
- note removed: "══ REGION POWER ══"
- note removed: "══ REGION SDI IN (Antmicro path — condensed) ══"
- note removed: "══ REGION SDI PLAYBACK OUT (from archive 07 — real symbols) ══"
- note removed: "══ REGION USB PHONE ══"
- title: LivCast Capture — Complete -> LivCast Capture - Complete
