File: kicad/LivCast_Capture.kicad_sch (KiCad schematic)
At the start: 13 parts, among them J101 Conn_DTAP, J102 Conn_USB_C_PWR, J201 Conn_USB_C_DATA, J701 Conn_HDMI_A, J702 Conn_BNC_031-70526-21, U101 TPS25751D, U102 LM76003, U103 TPS62130A, U201 CM5_IO, U202 TPS25751D, U701 TMDS_BUF_1TO2, U702 IT66021FN, U703 GS2962A

Commit message: Simplify schematic symbols: hide pin names, split CM5, single VIDEO_BUS.
Remove dense parallel pin stacks that made the sheet unreadable.

Co-authored-by: Cursor <cursoragent@cursor.com>
Parts:
- removed J201: Conn_USB_C_DATA, symbol livcast-capture:Conn_USB_C_DATA
- removed J701: Conn_HDMI_A, symbol livcast-capture:Conn_HDMI_A
- removed J702: Conn_BNC_031-70526-21, symbol sdi-mipi-bridge:Conn_BNC_031-70526-21
- removed U201: CM5_IO, symbol livcast-capture:CM5_IO
- removed U202: TPS25751D, symbol livcast-capture:TPS25751D
- removed U701: TMDS_BUF_1TO2, symbol livcast-capture:TMDS_BUF_1TO2
- removed U702: IT66021FN, symbol livcast-capture:IT66021FN
- removed U703: GS2962A, symbol livcast-capture:GS2962A
- added J103: Conn_USB_C_DATA, symbol livcast-capture:Conn_USB_C_DATA
- added J201: Conn_HDMI_A, symbol livcast-capture:Conn_HDMI_A
- added J501: Conn_BNC_031-70526-21, sdi-mipi-bridge-footprints:Conn_BNC_031-70526-21, symbol sdi-mipi-bridge:Conn_BNC_031-70526-21
- added U201: CM5_PWR, symbol livcast-capture:CM5_PWR
- added U202: CM5_HDMI, symbol livcast-capture:CM5_HDMI
- added U203: CM5_CSI0, symbol livcast-capture:CM5_CSI0
- added U204: CM5_CSI1, symbol livcast-capture:CM5_CSI1
- added U205: CM5_CTRL, symbol livcast-capture:CM5_CTRL
- added U301: TMDS_BUF_1TO2, symbol livcast-capture:TMDS_BUF_1TO2
- added U401: IT66021FN, symbol livcast-capture:IT66021FN
- added U501: GS2962A, symbol livcast-capture:GS2962A
Connections:
- net +3V3_EN is gone; now on net FB_3V3: U103.2 (EN)
- net +5V_EN is gone; now on net FB_5V: U102.2 (EN)
- net +1V2: now also U401.20 (VS), U501.21 (VDD_A_3V3), U501.24 (GND2)
- net +1V8: now also U401.21 (DE)
- net +3V3: now also U101.3 (CC2), U103.8 (PG), U301.2 (IN_D0_N), U401.22 (VDD33), U501.22 (VDD_CD), U501.23 (GND1); no longer U101.5 (VIN_3V3), U103.7 (VOUT)
- net BOOT_3V3: now also U103.6 (SW); no longer U103.9 (BOOT)
- net BOOT_5V: now also U102.6 (SW); no longer U102.9 (BOOT)
- net CSI0_CK_N: now also U203.1 (CSI0_D0_P)
- net CSI0_CK_P: now also U203.2 (CSI0_D0_N)
- net CSI0_D0_N: now also U203.9 (CSI0_CK_P)
- net CSI0_D0_P: now also U203.10 (CSI0_CK_N)
- net CSI0_D1_N: now also U203.7 (CSI0_D3_P)
- net CSI0_D1_P: now also U203.8 (CSI0_D3_N)
- net CSI0_D2_N: now also U203.5 (CSI0_D2_P)
- net CSI0_D2_P: now also U203.6 (CSI0_D2_N)
- net CSI0_D3_N: now also U203.3 (CSI0_D1_P)
- net CSI0_D3_P: now also U203.4 (CSI0_D1_N)
- net CSI1_CK_N: now also U204.1 (CSI1_D0_P)
- net CSI1_CK_P: now also U204.2 (CSI1_D0_N)
- net CSI1_D0_N: now also U204.9 (CSI1_CK_P)
- net CSI1_D0_P: now also U204.10 (CSI1_CK_N)
- net CSI1_D1_N: now also U204.7 (CSI1_D3_P)
- net CSI1_D1_P: now also U204.8 (CSI1_D3_N)
- net CSI1_D2_N: now also U204.5 (CSI1_D2_P)
- net CSI1_D2_P: now also U204.6 (CSI1_D2_N)
- net CSI1_D3_N: now also U204.3 (CSI1_D1_P)
- net CSI1_D3_P: now also U204.4 (CSI1_D1_N)
- net DE: now also U401.23 (VDD18), U401.24 (VDD12), U401.25 (GND1), U401.26 (GND2), U401.27 (GND3), U501.12 (DVB_ASI), U501.13 (SDIN), U501.14 (SDOUT), U501.15 (SCLK), U501.16 (CS#)
- net FB_3V3: no longer U103.4 (FB)
- net FB_5V: no longer U102.4 (FB)
- net GND: now also J101.1 (VIN), J102.1 (VBUS), U101.8 (PP5V), J103.1 (VBUS), J201.1 (D0_P), J201.2 (D0_N), U201.3 (+5V_3), U201.4 (GND_1), U201.5 (GND_2), U301.1 (IN_D0_P), U401.17 (VIDEO_BUS), U401.18 (PCLK), U401.19 (HS), U501.17 (SDO), U501.18 (SDO#), U501.19 (VDD_CORE_1V2), U501.20 (VDD_IO); no longer J101.2 (GND), J102.4 (GND), U101.11 (GND2)
- net HDMI_RX_CK_N: now also U301.12 (OUTA_D0_P), U401.9 (HPD)
- net HDMI_RX_CK_P: now also U301.13 (OUTA_D0_N), U401.10 (DDC_SDA)
- net HDMI_RX_D0_N: now also U301.18 (OUTA_CK_P), U401.15 (I2C_SCL)
- net HDMI_RX_D0_P: now also U301.19 (OUTA_CK_N), U401.16 (INT#)
- net HDMI_RX_D1_N: now also U301.16 (OUTA_D2_P), U401.13 (RESET#)
- net HDMI_RX_D1_P: now also U301.17 (OUTA_D2_N), U401.14 (I2C_SDA)
- net HDMI_RX_D2_N: now also U301.14 (OUTA_D1_P), U401.11 (DDC_SCL)
- net HDMI_RX_D2_P: now also U301.15 (OUTA_D1_N), U401.12 (+5V_HDMI)
- net HDMI_TX_CK_N: now also U202.1 (HDMI_TX_D0_P), U301.4 (IN_D1_N)
- net HDMI_TX_CK_P: now also U202.2 (HDMI_TX_D0_N), U301.5 (IN_D2_P)
- net HDMI_TX_D0_N: now also U202.7 (HDMI_TX_CK_P), U301.10 (VDD)
- net HDMI_TX_D0_P: now also U202.8 (HDMI_TX_CK_N), U301.11 (GND)
- net HDMI_TX_D1_N: now also U202.5 (HDMI_TX_D2_P), U301.8 (IN_CK_N)
- net HDMI_TX_D1_P: now also U202.6 (HDMI_TX_D2_N), U301.9 (OE#)
- net HDMI_TX_D2_N: now also U202.3 (HDMI_TX_D1_P), U301.6 (IN_D2_N)
- net HDMI_TX_D2_P: now also U202.4 (HDMI_TX_D1_N), U301.7 (IN_CK_P)
- net I2C_SCL: now also U101.1 (VBUS), U205.8 (SDI_TX_SPI_SCK), U401.2 (RX0_N); no longer U101.7 (I2C_SCL)
- net I2C_SDA: now also U101.2 (CC1), U205.9 (SDI_TX_SPI_CS), U401.3 (RX1_P); no longer U101.6 (I2C_SDA)
- net PD_GPIO1: now also U101.9 (PPHV); no longer U101.10 (GPIO1)
- net PG_3V3: now also U103.7 (VOUT); no longer U103.8 (PG)
- net PG_5V: now also U102.7 (VOUT); no longer U102.8 (PG)
- net SDI_TX_N: now also U501.25 (GND3)
- net SDI_TX_P: now also J501.1, U501.26 (GND4)
- net SDI_TX_SPI_CS: now also U205.1 (I2C_SDA), U501.1 (VIDEO_BUS)
- net SDI_TX_SPI_MOSI: now also U205.3 (SPI_MOSI), U501.4 (V_VSYNC)
- net SDI_TX_SPI_SCK: now also U205.2 (I2C_SCL), U501.2 (PCLK)
- net SPI_CS: now also U205.4 (SPI_MISO)
- net SPI_MISO: now also U205.6 (SPI_CS)
- net SPI_MOSI: now also U205.7 (SDI_TX_SPI_MOSI)
- net SPI_SCK: now also U205.5 (SPI_SCK)
- net SS_3V3: now also U103.1 (VIN); no longer U103.5 (SS)
- net SS_5V: now also U102.1 (VIN); no longer U102.5 (SS)
- net SW_3V3: now also U103.9 (BOOT); no longer U103.6 (SW)
- net SW_5V: now also U102.9 (BOOT); no longer U102.6 (SW)
- net USB_DN: now also J103.4 (CC1), U201.1 (+5V_1)
- net USB_DP: now also J103.5 (CC2), U201.2 (+5V_2)
- net VIN_RAW: now also J101.2 (GND), U102.5 (SS); no longer J101.1 (VIN), U101.9 (PPHV), U102.1 (VIN)
- removed net +5V0: U101.8 (PP5V), U102.7 (VOUT), U103.1 (VIN)
- net CC1_IN renamed CC2_PWR
- net CC2_PWR: now also U101.5 (VIN_3V3); no longer U101.2 (CC1)
- net CC2_IN renamed CC1_PWR
- net CC1_PWR: now also U101.6 (I2C_SDA); no longer U101.3 (CC2)
- removed net VBUS_IN: J102.1 (VBUS), U101.1 (VBUS)
- new net +5V: U102.8 (PG), U103.5 (SS), U201.6 (GND_3), U201.7 (USB_DP), U201.8 (USB_DN)
- new net +5V_HDMI: J201.3 (D1_P), U401.5 (RX2_P)
- new net BIT20_10: U501.9 (RATE_SEL0)
- new net BUCK33_EN: U103.4 (FB)
- new net BUCK_EN: U102.4 (FB)
- new net CC1_DATA: J103.3 (USB_DN)
- new net CC2_DATA: J103.2 (USB_DP)
- new net DVB_ASI: U501.5 (F_DE)
- new net GS_SDOUT: U501.3 (H_HSYNC)
- new net GS_STANDBY#: U501.10 (RATE_SEL1)
- new net HDMI_MON_CK_N: J201.7 (CK_P), U301.20 (OUTB_D0_P)
- new net HDMI_MON_CK_P: J201.8 (CK_N), U301.21 (OUTB_D0_N)
- new net HDMI_MON_D0_N: J201.13 (GND), U301.26 (OUTB_CK_P)
- new net HDMI_MON_D0_P: J201.14 (SHIELD), U301.27 (OUTB_CK_N)
- new net HDMI_MON_D1_N: J201.11 (HPD), U301.24 (OUTB_D2_P)
- new net HDMI_MON_D1_P: J201.12 (+5V), U301.25 (OUTB_D2_N)
- new net HDMI_MON_D2_N: J201.9 (DDC_SDA), U301.22 (OUTB_D1_P)
- new net HDMI_MON_D2_P: J201.10 (DDC_SCL), U301.23 (OUTB_D1_N)
- new net HDMI_MON_DDC_SCL: J201.5 (D2_P)
- new net HDMI_MON_DDC_SDA: J201.6 (D2_N)
- new net HDMI_MON_HPD: J201.4 (D1_N)
- new net HDMI_RX_DDC_SCL: U401.6 (RX2_N)
- new net HDMI_RX_DDC_SDA: U401.7 (RXC_P)
- new net HDMI_RX_HPD: U401.8 (RXC_N)
- new net IT66021_INT#: U401.1 (RX0_P)
- new net IT66021_RESET#: U401.4 (RX1_N)
- new net PP5V: U101.11 (GND2)
- new net PPHV: U101.10 (GPIO1)
- new net RATE_SEL0: U501.8 (BIT20_10)
- new net RATE_SEL1: U501.7 (STANDBY#)
- new net SDO_EN: U501.11 (SMPTE_BYPASS)
- new net SMPTE_BYPASS: U501.6 (SDO_EN)
- new net TMDS_OE#: U301.3 (IN_D1_P)
- new net VBUS: J102.4 (GND), J103.6 (GND), U101.7 (I2C_SCL)
Other:
- note added: "LivCast Capture Rev A — sparse symbols, pin names hidden, VIDEO_BUS simplified"
- note added: "Power column left. Labels on wire stubs only. CM5 split: U201-U205."
- note added: "SDI playback: CM5_HDMI -> TMDS 1:2 -> HDMI mon + IT66021FN -> VIDEO_BUS -> GS2962A -> BNC"
- note added: "VIDEO_BUS = 20-bit parallel PDATA/DIN — expand as bus on PCB (not drawn pin-by-pin)"
- note removed: "CM5 I/O"
- note removed: "HDMI OUT (monitor)"
- note removed: "HDMI TMDS (CM5 -> buffer)"
- note removed: "HDMI to IT66021FN"
- note removed: "LCD / DSI - TBD (archive_sheets/06)"
- note removed: "LivCast Capture - Complete (single sheet, Rev A)"
- note removed: "POWER"
- note removed: "Power column left. Labels on wire stubs >=10mm from pins. Ingest TBD: archive_sheets + README.md"
- note removed: "Rails"
- note removed: "Rule: never place net labels on pin bodies."
- note removed: "SDI OUT"
- note removed: "SDI playback: CM5 HDMI TX -> TMDS 1:2 -> HDMI mon + IT66021FN -> VIDEO[19:0] bus -> GS2962A -> BNC"
- note removed: "USB-C phone (network video)"
- note removed: "VIDEO[19:0] parallel bus"

Commit message: Redraw schematic with wire-only IC links and no stacked pin labels.
Adjacent HDMI/SDI chips connect by wires; labels only on power and region exits.

Co-authored-by: Cursor <cursoragent@cursor.com>
Connections:
- net CSI0_CK_P is gone; now on net CSI0_CK_N: U203.2 (CSI0_D0_N)
- net CSI0_D0_P is gone; now on net CSI0_D0_N: U203.10 (CSI0_CK_N)
- net CSI0_D1_N is gone; now on net CSI0_D0_N: U203.7 (CSI0_D3_P)
- net CSI0_D1_P is gone; now on net CSI0_D0_N: U203.8 (CSI0_D3_N)
- net CSI0_D3_N is gone; now on net CSI0_CK_N: U203.3 (CSI0_D1_P)
- net CSI0_D3_P is gone; now on net CSI0_CK_N: U203.4 (CSI0_D1_N)
- net CSI1_CK_P is gone; now on net CSI1_CK_N: U204.2 (CSI1_D0_N)
- net CSI1_D0_P is gone; now on net CSI1_D0_N: U204.10 (CSI1_CK_N)
- net CSI1_D1_N is gone; now on net CSI1_D0_N: U204.7 (CSI1_D3_P)
- net CSI1_D1_P is gone; now on net CSI1_D0_N: U204.8 (CSI1_D3_N)
- net CSI1_D3_N is gone; now on net CSI1_CK_N: U204.3 (CSI1_D1_P)
- net CSI1_D3_P is gone; now on net CSI1_CK_N: U204.4 (CSI1_D1_N)
- net HDMI_MON_CK_P is gone; now on an unnamed net: J201.8 (CK_N), U301.21 (OUTB_D0_N)
- net HDMI_MON_D0_N is gone; now on an unnamed net: J201.13 (GND), U301.26 (OUTB_CK_P)
- net HDMI_MON_D0_P is gone; now on an unnamed net: J201.14 (SHIELD), U301.27 (OUTB_CK_N)
- net HDMI_MON_D1_N is gone; now on an unnamed net: J201.11 (HPD), U301.24 (OUTB_D2_P)
- net HDMI_MON_D1_P is gone; now on an unnamed net: J201.12 (+5V), U301.25 (OUTB_D2_N)
- net HDMI_MON_D2_N is gone; now on an unnamed net: J201.9 (DDC_SDA), U301.22 (OUTB_D1_P)
- net HDMI_MON_D2_P is gone; now on an unnamed net: J201.10 (DDC_SCL), U301.23 (OUTB_D1_N)
- net HDMI_RX_CK_P is gone; now on an unnamed net: U301.13 (OUTA_D0_N), U401.10 (DDC_SDA)
- net HDMI_RX_D0_N is gone; now on an unnamed net: U301.18 (OUTA_CK_P), U401.15 (I2C_SCL)
- net HDMI_RX_D0_P is gone; now on an unnamed net: U301.19 (OUTA_CK_N), U401.16 (INT#)
- net HDMI_RX_D1_N is gone; now on an unnamed net: U301.16 (OUTA_D2_P), U401.13 (RESET#)
- net HDMI_RX_D1_P is gone; now on an unnamed net: U301.17 (OUTA_D2_N), U401.14 (I2C_SDA)
- net HDMI_RX_D2_N is gone; now on an unnamed net: U301.14 (OUTA_D1_P), U401.11 (DDC_SCL)
- net HDMI_RX_D2_P is gone; now on an unnamed net: U301.15 (OUTA_D1_N), U401.12 (+5V_HDMI)
- net HDMI_TX_CK_P is gone; now on an unnamed net: U202.2 (HDMI_TX_D0_N), U301.5 (IN_D2_P)
- net HDMI_TX_D0_N is gone; now on an unnamed net: U202.7 (HDMI_TX_CK_P), U301.10 (VDD)
- net HDMI_TX_D0_P is gone; now on an unnamed net: U202.8 (HDMI_TX_CK_N), U301.11 (GND)
- net HDMI_TX_D1_N is gone; now on an unnamed net: U202.5 (HDMI_TX_D2_P), U301.8 (IN_CK_N)
- net HDMI_TX_D1_P is gone; now on an unnamed net: U202.6 (HDMI_TX_D2_N), U301.9 (OE#)
- net HDMI_TX_D2_N is gone; now on an unnamed net: U202.3 (HDMI_TX_D1_P), U301.6 (IN_D2_N)
- net HDMI_TX_D2_P is gone; now on an unnamed net: U202.4 (HDMI_TX_D1_N), U301.7 (IN_CK_P)
- net I2C_SDA is gone; now on net I2C_SCL: U101.2 (CC1), U205.9 (SDI_TX_SPI_CS), U401.3 (RX1_P)
- net SDI_TX_SPI_MOSI is gone; now on net SDI_TX_SPI_CS: U205.3 (SPI_MOSI), U501.4 (V_VSYNC)
- net SDI_TX_SPI_SCK is gone; now on net SDI_TX_SPI_CS: U205.2 (I2C_SCL), U501.2 (PCLK)
- net SPI_CS is gone; now on net SDI_TX_SPI_CS: U205.4 (SPI_MISO)
- net SPI_MISO is gone; now on net I2C_SCL: U205.6 (SPI_CS)
- net SPI_MOSI is gone; now on net I2C_SCL: U205.7 (SDI_TX_SPI_MOSI)
- net DE: no longer U401.23 (VDD18), U401.24 (VDD12), U401.25 (GND1), U401.26 (GND2), U401.27 (GND3), U501.12 (DVB_ASI), U501.13 (SDIN), U501.14 (SDOUT), U501.15 (SCLK), U501.16 (CS#)
- net HDMI_MON_CK_N: no longer names the net of J201.7 (CK_P), U301.20 (OUTB_D0_P)
- net HDMI_RX_CK_N: no longer names the net of U301.12 (OUTA_D0_P), U401.9 (HPD)
- net HDMI_TX_CK_N: no longer names the net of U202.1 (HDMI_TX_D0_P), U301.4 (IN_D1_N)
- net SDI_TX_P: no longer names the net of J501.1, U501.26 (GND4)
- new net: U401.23 (VDD18), U401.24 (VDD12), U401.25 (GND1), U401.26 (GND2), U401.27 (GND3), U501.12 (DVB_ASI), U501.13 (SDIN), U501.14 (SDOUT), U501.15 (SCLK), U501.16 (CS#)
Other:
- note added: "LivCast Capture Rev A — wire-only IC links; labels on power / region exits only"
- note added: "Playback row: CM5_HDMI -wires-> TMDS -OUTA wires-> HDMI mon; OUTB wires-> IT66021 -VIDEO_BUS-> GS2962 -> BNC"
- note added: "VIDEO_BUS = 20-bit parallel (single wire on schematic). CSI/CTRL globals pitched 15mm on long stubs."
- note added: "to monitor"
- note removed: "LivCast Capture Rev A — sparse symbols, pin names hidden, VIDEO_BUS simplified"
- note removed: "Power column left. Labels on wire stubs only. CM5 split: U201-U205."
- note removed: "SDI playback: CM5_HDMI -> TMDS 1:2 -> HDMI mon + IT66021FN -> VIDEO_BUS -> GS2962A -> BNC"
- note removed: "VIDEO_BUS = 20-bit parallel PDATA/DIN — expand as bus on PCB (not drawn pin-by-pin)"

Commit message: Replace dense pin schematic with a readable block diagram.
Archive the auto-generated pin dump; keep one clear architecture sheet.

Co-authored-by: Cursor <cursoragent@cursor.com>
Parts:
- removed J101: Conn_DTAP, symbol livcast-capture:Conn_DTAP
- removed J102: Conn_USB_C_PWR, symbol livcast-capture:Conn_USB_C_PWR
- removed J103: Conn_USB_C_DATA, symbol livcast-capture:Conn_USB_C_DATA
- removed J201: Conn_HDMI_A, symbol livcast-capture:Conn_HDMI_A
- removed J501: Conn_BNC_031-70526-21, sdi-mipi-bridge-footprints:Conn_BNC_031-70526-21, symbol sdi-mipi-bridge:Conn_BNC_031-70526-21
- removed U101: TPS25751D, symbol livcast-capture:TPS25751D
- removed U102: LM76003, symbol livcast-capture:LM76003
- removed U103: TPS62130A, symbol livcast-capture:TPS62130A
- removed U201: CM5_PWR, symbol livcast-capture:CM5_PWR
- removed U202: CM5_HDMI, symbol livcast-capture:CM5_HDMI
- removed U203: CM5_CSI0, symbol livcast-capture:CM5_CSI0
- removed U204: CM5_CSI1, symbol livcast-capture:CM5_CSI1
- removed U205: CM5_CTRL, symbol livcast-capture:CM5_CTRL
- removed U301: TMDS_BUF_1TO2, symbol livcast-capture:TMDS_BUF_1TO2
- removed U401: IT66021FN, symbol livcast-capture:IT66021FN
- removed U501: GS2962A, symbol livcast-capture:GS2962A
- added J_DTAP: Conn_DTAP, symbol livcast-capture:Conn_DTAP
- added J_HDMI_IN, J_HDMI_OUT: Conn_HDMI_A, symbol livcast-capture:Conn_HDMI_A
- added J_SDI_IN, J_SDI_OUT: BNC, symbol sdi-mipi-bridge:Conn_BNC_031-70526-21
- added J_USBC_PHONE: Conn_USB_C_DATA, symbol livcast-capture:Conn_USB_C_DATA
- added J_USBC_PWR: Conn_USB_C_PWR, symbol livcast-capture:Conn_USB_C_PWR
Other:
- note added: "(40-pin FFC)"
- note added: "(playback, not loop)"
- note added: "+ CrossLink CSI"
- note added: "3.5 inch SPI preview"
- note added: "5V / 3V3 REGULATORS"
- note added: "5V buck + 3V3 LDO"
- note added: "720p / 1080i / 1080p"
- note added: "Antmicro-class path"
- note added: "CM5"
- note added: "CM5 + bridges"
- note added: "CSI0 / CSI1 ingest"
- note added: "Compute Module 5"
- note added: "D-Tap + USB-C PD"
- note added: "GS2962A path"
- note added: "HDMI IN / IT6616"
- note added: "HDMI OUT + SDI PLAY"
- note added: "HDMI to MIPI CSI"
- note added: "Hosyond 480x320"
- note added: "IT66021 + GS2962A"
- note added: "J_LCD"
- note added: "LCD 40-pin"
- note added: "Legend: yellow boxes = blocks | mid-wire labels = nets | edge J* = connectors"
- note added: "LivCast Capture - Block Schematic (Rev A)"
- note added: "POWER IN"
- note added: "Readable architecture sheet. Dense pin sch archived as LivCast_Capture_dense_pins.kicad_sch"
- note added: "SDI IN / GS2971A"
- note added: "USB gadget + HDMI TX"
- note added: "USB-C PHONE"
- note added: "battery / wall"
- note added: "data + charge"
- note added: "monitor + SDI deck"
- note removed: "HDMI IN ingest - TBD (archive_sheets/03)"
- note removed: "LivCast Capture Rev A — wire-only IC links; labels on power / region exits only"
- note removed: "Playback row: CM5_HDMI -wires-> TMDS -OUTA wires-> HDMI mon; OUTB wires-> IT66021 -VIDEO_BUS-> GS2962 -> BNC"
- note removed: "SDI IN ingest - TBD (archive_sheets/04, Antmicro)"
- note removed: "VIDEO_BUS = 20-bit parallel (single wire on schematic). CSI/CTRL globals pitched 15mm on long stubs."
- note removed: "to monitor"
- title: LivCast Capture - Complete -> LivCast Capture - Block Schematic (Rev A)
